File: Controller/HW/KiCad_Files/Controller.kicad_pcb (KiCad board)
At the start: 4 copper layers, 70 x 70 mm, 79 parts, among them J1 Groove, J2 USB, J3 JTAG, J4 Speaker, J5 Driver, J6 QWIIC, Q1 Q_NPN_BEC, Q2 Q_NPN_BEC, Q3 Q_NPN_BEC, Q4 Q_NMOS_GSD, Q5 Q_NMOS_GSD, SW1 Reset, SW2 Config, SW3 SW_Coded, U1 USBLC6-2SC6, U2 CP2102N-Axx-xQFN28, U3 ESP32-S3-WROOM-1, U4 MAX98357A, U5 AP1117-33

Commit message: PCB Zwischenstand
Parts:
- added D2: Power, LED_SMD:LED_0805_2012Metric, F.Cu at (212.8, 90.8)
- added D3: TX, LED_SMD:LED_0805_2012Metric, F.Cu at (182.8, 32.8)
- added D4: RX, LED_SMD:LED_0805_2012Metric, F.Cu at (182.8, 35.9)
- added R1: 1k, Resistor_SMD:R_0805_2012Metric, F.Cu at (212.7, 93.8)
- added R10: 1k, Resistor_SMD:R_0805_2012Metric, F.Cu at (187.2, 32.8)
- added R11: 1k, Resistor_SMD:R_0805_2012Metric, F.Cu at (187.2, 35.7)
- D1: renamed from D3; value RB751V40 -> NSR0320
- D13: renamed from D18; value RB751V40 -> NSR0320
- Q1, Q2, Q3: value Q_NPN_BEC -> MMBT3904
- Q4, Q5: value Q_NMOS_GSD -> NX138AK
- R4: renamed from R8; value 10k -> 1k
- moved C11 59.9 mm to (278.2, 38.7)
- moved D18 59.9 mm to (277.8, 33.7)
- moved D19 59.9 mm to (277.8, 35.7)
- moved Q4 59.9 mm to (273.8, 33.2)
- moved Q5 59.9 mm to (273.8, 36.7)
- moved R26 59.9 mm to (270.8, 33.2)
- moved R27 59.9 mm to (270.8, 36.7)
- moved R28 59.9 mm to (275.2, 30.2)
- moved R29 59.9 mm to (275.2, 39.7)
- moved Q3 43.1 mm to (252.7, 33.4)
- moved R21 43.1 mm to (248.9, 29.4)
- moved R22 43.1 mm to (248.6, 32.2)
- moved J6 31.8 mm to (228.8, 64.8)
- moved R23 25.0 mm to (233.8, 17.3)
- moved Q1 21.6 mm to (198.2, 32.8)
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- renumbered C11 to C1, C8 to C11, C9 to C12, C12 to C2, C1 to C3, C2 to C4, C4 to C5, C3 to C6, C5 to C7, C6 to C8, C7 to C9, D11 to D10, D12 to D11, D13 to D12, D7 to D18, D8 to D19, D9 to D20, D10 to D21, D1 to D5, D2 to D6, D4 to D7, D5 to D8, D6 to D9, J2 to J1, J3 to J2, J4 to J3, J5 to J4, J1 to J5, R16 to R12, R15 to R13, R13 to R15, R12 to R16, R11 to R17, R17 to R18, R18 to R19, R3 to R2, R19 to R20, R20 to R21, R24 to R23, R1 to R24, R2 to R25, R21 to R26, R25 to R27, R23 to R28, R26 to R29, R4 to R3, R9 to R8, R10 to R9, SW2 to SW1, SW1 to SW2, U5 to U1, U1 to U2, U2 to U3, U3 to U4, U4 to U5
Connections:
- J3 pad 1: Net-(J4-Pin_1) -> Net-(J3-Pin_1)
- J3 pad 2: Net-(J4-Pin_2) -> Net-(J3-Pin_2)
- U3 pad 18: unconnected-(U2-~{RXT}/GPIO.1-Pad18) -> Net-(D4-K)
- U3 pad 19: unconnected-(U2-~{TXT}/GPIO.0-Pad19) -> Net-(D3-K)
- U5 pad 10: Net-(J4-Pin_2) -> Net-(J3-Pin_1)
- U5 pad 9: Net-(J4-Pin_1) -> Net-(J3-Pin_2)
Routing:
- net GND: track 52.4 -> 80.1 mm, vias 29 -> 46
- net /ESP32/Rst: track 50.7 -> 40.7 mm, vias 2 -> 1
- net +5V: track 18.6 -> 28.6 mm
- net /ESP32/RX_Driver: track 0.00 -> 6.91 mm
- net /ESP32/Controller_Interrupt: track 0.00 -> 6.91 mm
- net /ESP32/TX_Driver: track 0.00 -> 6.91 mm
- net /ESP32/Driver_Interrupt: track 0.00 -> 6.89 mm
- net Net-(J3-Pin_2): track 0.00 -> 6.87 mm
- net Net-(J3-Pin_1): track 0.00 -> 6.87 mm
- net /Audio/LRCLK: track 0.00 -> 3.37 mm
- net /Audio/BCLK: track 0.00 -> 2.67 mm
- net Net-(Q1-B): track 5.64 -> 3.66 mm
- net /ESP32/Boot: track 1.62 -> 0.00 mm
- removed copper zone on B.Cu, net GND
- removed copper zone on F.Cu, net GND

Commit message: Controller Rev 1 PCB fertig
Parts:
- added G***: LOGO, LOGO, F.Cu at (153.1, 81.9)
- SW1: value Config -> ESP Config
- SW3: value SW_Coded -> Gain
- moved R21 146.7 mm to (138.6, 126.2), turned to 90 degrees
- moved Q3 144.5 mm to (141.9, 126.2)
- moved R23 125.3 mm to (167.8, 123.9)
- moved R22 120.8 mm to (167.8, 121.9), turned to 180 degrees
- moved SW3 115.4 mm to (156.8, 123.4)
- moved Q4 114.5 mm to (165.8, 71.4)
- moved Q5 114.5 mm to (165.8, 74.9)
- moved R26 114.5 mm to (162.8, 71.4)
- moved R27 114.5 mm to (162.8, 74.9)
- moved R28 113.1 mm to (168.8, 68.4)
- moved R29 113.1 mm to (168.8, 77.9)
- moved C11 112.1 mm to (172.8, 77.0)
- moved D18 112.1 mm to (172.3, 71.9)
- moved D19 112.1 mm to (172.3, 73.9)
- moved C8 89.6 mm to (167.8, 119.9)
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Connections:
- J3 pad MP: (no net) -> GND
- J6 pad MP: (no net) -> GND
- R22 pad 1: +3.3V -> +5V
- SW1 pad 4: /ESP32/LOG -> /ESP32/JTAG
- SW1 pad 6: /ESP32/JTAG -> /ESP32/LOG
Routing:
- net +3.3V: track 38.4 -> 209.3 mm, vias 0 -> 9
- net +5V: track 28.6 -> 160.2 mm, vias 2 -> 7
- net /ESP32/SCL: track 0.00 -> 88.2 mm, vias 0 -> 4
- net /ESP32/SDA: track 0.00 -> 85.1 mm, vias 0 -> 2
- net GND: track 80.1 -> 24.2 mm, vias 46 -> 400
- net /ESP32/TX_Driver: track 6.91 -> 59.5 mm
- net /Audio/LRCLK: track 3.37 -> 49.6 mm
- net /Audio/BCLK: track 2.67 -> 47.3 mm
- net /Audio/DIN: track 0.00 -> 42.7 mm, vias 0 -> 2
- net /ESP32/Boot: track 0.00 -> 42.3 mm, vias 0 -> 2
- net /ESP32/RX_Driver: track 6.91 -> 44.9 mm
- net Net-(Q3-C): track 0.00 -> 31.1 mm
- net /ESP32/Controller_Interrupt: track 6.91 -> 37.9 mm
- net /ESP32/Driver_Interrupt: track 6.89 -> 37.5 mm
- net Net-(D3-K): track 0.00 -> 29.5 mm
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- added copper zone on B.Cu, net GND
- added copper zone on F.Cu, net GND
Other:
- outline, holes or cut-outs redrawn
- board text added: "0: 6dB 1: 9dB 2: 12dB 3: 15dB"
- board text added: "AÜP 2023 High5Dynamics Controller Rev 1"
- board text added: "JTAG"
- board text added: "LOG"
- board text added: "VSPI"

Commit message: BOM update
Parts:
- moved G*** 0.42 mm to (153.5, 81.9)
Changed lines of the file:
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@@
   )
   (footprint "LOGO" (layer "F.Cu")
-    (at 153.08 81.905)
+    (at 153.5 81.905)
     (attr board_only exclude_from_pos_files exclude_from_bom)
     (fp_text reference "G***" (at 0 0) (layer "F.SilkS") hide
