File: Controller/HW/KiCad_Files/Audio.kicad_sch (KiCad schematic)
At the start: 10 parts, among them J4 Speaker, Q1 Q_NPN_BEC, SW3 SW_Coded, U4 MAX98357A

Commit message: PCB Zwischenstand
Parts:
- J3: renamed from J4; DigiKey (none) -> 455-2872-1-ND; MPN B2B-PH-SM4-TB(LF)(SN) -> B2B-PH-SM4-TBT(LF)(SN)
- Q1: value Q_NPN_BEC -> MMBT3904; DigiKey (none) -> 1727-4044-1-ND
- U5: renamed from U4; DigiKey (none) -> MAX98357AETE+TCT-ND
- renumbered R24 to R23
Connections:
- net at U5.10 (OUTN): now also J3.1 (Pin_1); no longer J3.2 (Pin_2)
- net at U5.9 (OUTP): now also J3.2 (Pin_2); no longer J3.1 (Pin_1)

Commit message: Controller Rev 1 PCB fertig
Parts:
- SW3: value SW_Coded -> Gain
Connections:
- net +3.3V is gone; now on net +5V: R22.1
- net GND: now also J3.MP

Commit message: BOM update
Parts:
- C2: DigiKey (none) -> 1276-2449-1-ND
- C3: DigiKey (none) -> 1276-1096-1-ND
- R22, R9: DigiKey (none) -> CR0805-FX-1002ELFCT-ND
- R23: DigiKey (none) -> CR0805-FX-1003ELFCT-ND
Changed lines of the file:
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@@
+      (effects (font (size 1.27 1.27)) hide)
+    )
+    (property "DigiKey" "CR0805-FX-1002ELFCT-ND" (at 92.71 129.54 0)
       (effects (font (size 1.27 1.27)) hide)
     )
@@
     )
     (property "Datasheet" "~" (at 156.21 86.36 0)
+      (effects (font (size 1.27 1.27)) hide)
+    )
+    (property "DigiKey" "1276-2449-1-ND" (at 156.21 86.36 0)
       (effects (font (size 1.27 1.27)) hide)
     )
@@
       (effects (font (size 1.27 1.27)) hide)
     )
+    (property "DigiKey" "CR0805-FX-1003ELFCT-ND" (at 95.25 93.98 0)
+      (effects (font (size 1.27 1.27)) hide)
+    )
     (pin "1")
     (pin "2")
@@
     )
     (property "Datasheet" "~" (at 135.89 86.36 0)
+      (effects (font (size 1.27 1.27)) hide)
+    )
+    (property "DigiKey" "1276-1096-1-ND" (at 135.89 86.36 0)
       (effects (font (size 1.27 1.27)) hide)
     )
@@
       (effects (font (size 1.27 1.27)) hide)
     )
+    (property "DigiKey" "1276-2449-1-ND" (at 146.05 86.36 0)
+      (effects (font (size 1.27 1.27)) hide)
+    )
     (pin "1")
     (pin "2")
@@
       (effects (font (size 1.27 1.27)) hide)
     )
+    (property "DigiKey" "CR0805-FX-1002ELFCT-ND" (at 80.01 140.97 0)
+      (effects (font (size 1.27 1.27)) hide)
+    )

Commit message: Schemas aktualisiert mit PDF
Other:
- company: (none) -> High5Dynamics
- title: (none) -> Controller
Changed lines of the file:
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@@
 (kicad_sch (version 20230121) (generator eeschema)
   (paper "A4")
+  (title_block
+    (title "Controller")
+    (date "2023-05-07")
+    (rev "1")
+    (company "High5Dynamics")
+  )
   (junction (at 135.89 81.28) (diameter 0) (color 0 0 0 0)
   )
@@
     )
     (pin "1")
+    (pin "2")
     (pin "MP")
-    (pin "2")
-    (instances
-      (project "Controller"
+    (instances
+      (project "Controller"
