File: Controller/HW/KiCad_Files/ESP32.kicad_sch (KiCad schematic)
At the start: 24 parts, among them J3 JTAG, SW1 Reset, SW2 Config, U3 ESP32-S3-WROOM-1

Commit message: PCB Zwischenstand
Parts:
- D13: renamed from D18; value RB751V40 -> NSR0320; DigiKey 1727-6301-1-ND -> NSR0320MW2T3GOSCT-ND
- U4: renamed from U3; DigiKey (none) -> 1965-ESP32-S3-WROOM-1-N8CT-ND
- renumbered C4 to C5, C3 to C6, D1 to D5, D2 to D6, D4 to D7, D5 to D8, J3 to J2, R16 to R12, R15 to R13, R13 to R15, R12 to R16, R11 to R17, R17 to R18, R18 to R19, R19 to R20, SW2 to SW1, SW1 to SW2

Commit message: Controller Rev 1 PCB fertig
Parts:
- SW1: value Config -> ESP Config
Connections:
- net JTAG: now also SW1.4; no longer SW1.6
- net LOG: now also SW1.6; no longer SW1.4
Changed lines of the file:
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@@
     )
   )
-  (symbol (lib_id "Switch:SW_DIP_x03") (at 33.02 96.52 0) (unit 1)
+  (symbol (lib_id "Switch:SW_DIP_x03") (at 33.02 91.44 0) (mirror x) (unit 1)
     (in_bom yes) (on_board yes) (dnp no)
     (property "Reference" "SW1" (at 33.02 87.63 0)
       (effects (font (size 1.27 1.27)))
     )
-    (property "Value" "Config" (at 33.02 100.33 0)
+    (property "Value" "ESP Config" (at 33.02 100.33 0)
       (effects (font (size 1.27 1.27)))
     )
-    (property "Footprint" "Button_Switch_SMD:SW_DIP_SPSTx03_Slide_Omron_A6S-310x_W8.9mm_P2.54mm" (at 33.02 96.52 0)
+    (property "Footprint" "Button_Switch_SMD:SW_DIP_SPSTx03_Slide_Omron_A6S-310x_W8.9mm_P2.54mm" (at 33.02 91.44 0)
       (effects (font (size 1.27 1.27)) hide)
     )
-    (property "Datasheet" "~" (at 33.02 96.52 0)
+    (property "Datasheet" "~" (at 33.02 91.44 0)
       (effects (font (size 1.27 1.27)) hide)
     )
-    (property "MPN" "DS04-254-2-03BK-SMT" (at 26.67 102.87 0)
+    (property "MPN" "DS04-254-2-03BK-SMT" (at 26.67 85.09 0)
       (effects (font (size 1.27 1.27)) hide)
     )

Commit message: BOM update
Parts:
- C5: DigiKey (none) -> 1276-1026-1-ND
- C6: DigiKey (none) -> 1276-1096-1-ND
- D14, D15, D16, D17: DigiKey D1213A-01WS-7 -> D1213A-01WS-7DICT-ND
- D5, D7, D8: DigiKey (none) -> 475-1410-1-ND
- D6: DigiKey (none) -> 475-1278-1-ND
- J2: DigiKey (none) -> 1175-1629-ND; MPN 3221-10-0300-00 -> 3220-10-0300-00
- R12, R13, R14, R16: DigiKey (none) -> CR0805-FX-1002ELFCT-ND
- R15, R17, R18, R19, R20: DigiKey (none) -> CR0805-FX-1001ELFCT-ND
- SW1: DigiKey (none) -> 2223-DS04-254-2-03BK-SMT-ND
Changed lines of the file:
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@@
+      (effects (font (size 1.27 1.27)) hide)
+    )
+    (property "DigiKey" "CR0805-FX-1002ELFCT-ND" (at 55.88 48.26 0)
       (effects (font (size 1.27 1.27)) hide)
     )
@@
       (effects (font (size 1.27 1.27)) hide)
     )
+    (property "DigiKey" "475-1410-1-ND" (at 250.19 74.93 0)
+      (effects (font (size 1.27 1.27)) hide)
+    )
     (pin "1")
     (pin "2")
@@
       (effects (font (size 1.27 1.27)) hide)
     )
+    (property "DigiKey" "475-1410-1-ND" (at 219.71 74.93 0)
+      (effects (font (size 1.27 1.27)) hide)
+    )
     (pin "1")
     (pin "2")
@@
       (effects (font (size 1.27 1.27)) hide)
     )
+    (property "DigiKey" "CR0805-FX-1001ELFCT-ND" (at 265.43 66.04 0)
+      (effects (font (size 1.27 1.27)) hide)
+    )
     (pin "1")
     (pin "2")
@@
     )
     (property "Datasheet" "~" (at 219.71 66.04 0)
+      (effects (font (size 1.27 1.27)) hide)
+    )
+    (property "DigiKey" "CR0805-FX-1001ELFCT-ND" (at 219.71 66.04 0)
       (effects (font (size 1.27 1.27)) hide)
     )
@@
     )
     (property "Datasheet" "~" (at 265.43 74.93 0)
+      (effects (font (size 1.27 1.27)) hide)
+    )
+    (property "DigiKey" "475-1410-1-ND" (at 265.43 74.93 0)
       (effects (font (size 1.27 1.27)) hide)
     )
@@
       (effects (font (size 1.27 1.27)) hide)
     )
-    (property "DigiKey" "D1213A-01WS-7" (at 232.41 133.35 90)
+    (property "DigiKey" "D1213A-01WS-7DICT-ND" (at 232.41 133.35 90)
       (effects (font (size 1.27 1.27)) hide)
     )
@@
     )
     (property "Datasheet" "~" (at 52.07 101.6 0)
+      (effects (font (size 1.27 1.27)) hide)
+    )
+    (property "DigiKey" "CR0805-FX-1002ELFCT-ND" (at 52.07 101.6 0)
       (effects (font (size 1.27 1.27)) hide)
     )
@@
       (effects (font (size 1.27 1.27)) hide)
     )
+    (property "DigiKey" "CR0805-FX-1001ELFCT-ND" (at 48.26 53.34 0)
+      (effects (font (size 1.27 1.27)) hide)
+    )
     (pin "1")
     (pin "2")
@@
     )
     (property "MPN" "DS04-254-2-03BK-SMT" (at 26.67 85.09 0)
+      (effects (font (size 1.27 1.27)) hide)
+    )
+    (property "DigiKey" "2223-DS04-254-2-03BK-SMT-ND" (at 33.02 91.44 0)
       (effects (font (size 1.27 1.27)) hide)
     )
@@
       (effects (font (size 1.27 1.27)) hide)
     )
+    (property "DigiKey" "CR0805-FX-1002ELFCT-ND" (at 41.91 101.6 0)
+      (effects (font (size 1.27 1.27)) hide)
+    )
     (pin "1")
     (pin "2")
@@
     )
     (property "Datasheet" "~" (at 55.88 58.42 0)
+      (effects (font (size 1.27 1.27)) hide)
+    )
+    (property "DigiKey" "1276-1026-1-ND" (at 55.88 58.42 0)
       (effects (font (size 1.27 1.27)) hide)
     )
@@
       (effects (font (size 1.27 1.27)) hide)
     )
+    (property "DigiKey" "CR0805-FX-1001ELFCT-ND" (at 250.19 66.04 0)
+      (effects (font (size 1.27 1.27)) hide)
+    )
     (pin "1")
     (pin "2")
@@
       (effects (font (size 1.27 1.27)) hide)
     )
+    (property "DigiKey" "1276-1096-1-ND" (at 82.55 40.64 0)
+      (effects (font (size 1.27 1.27)) hide)
+    )
     (pin "1")
     (pin "2")
@@
       (effects (font (size 1.27 1.27)) hide)
     )
+    (property "DigiKey" "CR0805-FX-1002ELFCT-ND" (at 60.96 101.6 0)
+      (effects (font (size 1.27 1.27)) hide)
+    )
     (pin "1")
     (pin "2")
@@
       (effects (font (size 1.27 1.27)) hide)
     )
-    (property "DigiKey" "D1213A-01WS-7" (at 207.01 133.35 90)
+    (property "DigiKey" "D1213A-01WS-7DICT-ND" (at 207.01 133.35 90)
       (effects (font (size 1.27 1.27)) hide)
     )
@@
       (effects (font (size 1.27 1.27)) hide)
     )
-    (property "MPN" "3221-10-0300-00" (at 256.54 123.19 0)
+    (property "MPN" "3220-10-0300-00" (at 256.54 123.19 0)
+      (effects (font (size 1.27 1.27)) hide)
+    )
+    (property "DigiKey" "1175-1629-ND" (at 256.54 123.19 0)
       (effects (font (size 1.27 1.27)) hide)
     )
@@
       (effects (font (size 1.27 1.27)) hide)
     )
+    (property "DigiKey" "475-1278-1-ND" (at 234.95 74.93 0)
+      (effects (font (size 1.27 1.27)) hide)
+    )
     (pin "1")
     (pin "2")
@@
       (effects (font (size 1.27 1.27)) hide)
     )
-    (property "DigiKey" "D1213A-01WS-7" (at 219.71 133.35 90)
+    (property "DigiKey" "D1213A-01WS-7DICT-ND" (at 219.71 133.35 90)
       (effects (font (size 1.27 1.27)) hide)
     )
@@
       (effects (font (size 1.27 1.27)) hide)
     )
-    (property "DigiKey" "D1213A-01WS-7" (at 245.11 133.35 90)
+    (property "DigiKey" "D1213A-01WS-7DICT-ND" (at 245.11 133.35 90)
       (effects (font (size 1.27 1.27)) hide)
     )
@@
       (effects (font (size 1.27 1.27)) hide)
     )
+    (property "DigiKey" "CR0805-FX-1001ELFCT-ND" (at 234.95 66.04 0)
+      (effects (font (size 1.27 1.27)) hide)
+    )

Commit message: Schemas aktualisiert mit PDF
Other:
- company: (none) -> High5Dynamics
- title: (none) -> Controller
Changed lines of the file:
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@@
 (kicad_sch (version 20230121) (generator eeschema)
   (paper "A4")
+  (title_block
+    (title "Controller")
+    (date "2023-05-07")
+    (rev "1")
+    (company "High5Dynamics")
+  )
   (junction (at 60.96 91.44) (diameter 0) (color 0 0 0 0)
   )
