File: Controller/HW/KiCad_Files/Peripherals.kicad_sch (KiCad schematic)
At the start: 22 parts, among them J1 Driver, J1 Groove, J6 QWIIC, Q4 Q_NMOS_GSD, Q5 Q_NMOS_GSD

Commit message: PCB Zwischenstand
Parts:
- Q4, Q5: value Q_NMOS_GSD -> NX138AK
- renumbered D7 to D18, D8 to D19, D9 to D20, D10 to D21, J1 to J5, R1 to R24, R2 to R25, R21 to R26, R25 to R27, R23 to R28, R26 to R29
Other:
- moved on the sheet: C2, D20, D21, J6

Commit message: Controller Rev 1 PCB fertig
Connections:
- net GND: now also J5.MP, J6.MP
Changed lines of the file:
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@@
   (junction (at 153.67 54.61) (diameter 0) (color 0 0 0 0)
   )
+  (junction (at 173.99 110.49) (diameter 0) (color 0 0 0 0)
+  )
   (junction (at 175.26 46.99) (diameter 0) (color 0 0 0 0)
   )
@@
   )
   (junction (at 114.3 153.67) (diameter 0) (color 0 0 0 0)
+  )
+  (junction (at 139.7 163.83) (diameter 0) (color 0 0 0 0)
   )
   (junction (at 161.29 102.87) (diameter 0) (color 0 0 0 0)
@@
     (stroke (width 0) (type default))
   )
+  (wire (pts (xy 173.99 110.49) (xy 173.99 111.76))
+    (stroke (width 0) (type default))
+  )
   (wire (pts (xy 160.02 38.1) (xy 160.02 44.45))
     (stroke (width 0) (type default))
   )
   (wire (pts (xy 115.57 46.99) (xy 161.29 46.99))
+    (stroke (width 0) (type default))
+  )
+  (wire (pts (xy 173.99 110.49) (xy 173.99 107.95))
     (stroke (width 0) (type default))
   )
@@
     (stroke (width 0) (type default))
   )
+  (wire (pts (xy 139.7 163.83) (xy 139.7 161.29))
+    (stroke (width 0) (type default))
+  )
   (wire (pts (xy 115.57 90.17) (xy 115.57 91.44))
     (stroke (width 0) (type default))
@@
   )
   (wire (pts (xy 173.99 46.99) (xy 175.26 46.99))
+    (stroke (width 0) (type default))
+  )
+  (wire (pts (xy 139.7 163.83) (xy 140.97 163.83))
     (stroke (width 0) (type default))
   )
@@
     (stroke (width 0.25) (type dash))
   )
+  (wire (pts (xy 173.99 110.49) (xy 175.26 110.49))
+    (stroke (width 0) (type default))
+  )
   (wire (pts (xy 115.57 45.72) (xy 115.57 46.99))
     (stroke (width 0) (type default))
@@
     (stroke (width 0.25) (type dash))
   )
-  (wire (pts (xy 173.99 109.22) (xy 173.99 107.95))
-    (stroke (width 0) (type default))
-  )
   (polyline (pts (xy 110.49 30.48) (xy 110.49 73.66))
     (stroke (width 0.25) (type dash))
@@
     (stroke (width 0) (type default))
   )
-  (wire (pts (xy 139.7 162.56) (xy 139.7 161.29))
+  (wire (pts (xy 139.7 165.1) (xy 139.7 163.83))
     (stroke (width 0) (type default))
   )
@@
     )
   )
-  (symbol (lib_id "Connector_Generic:Conn_01x04") (at 180.34 102.87 0) (unit 1)
+  (symbol (lib_name "Conn_01x04_1") (lib_id "Connector_Generic:Conn_01x04") (at 180.34 102.87 0) (unit 1)
     (in_bom yes) (on_board yes) (dnp no)
     (property "Reference" "J5" (at 180.34 97.79 0)
       (effects (font (size 1.27 1.27)))
     )
-    (property "Value" "Groove" (at 180.34 110.49 0)
+    (property "Value" "Groove" (at 180.34 113.03 0)
       (effects (font (size 1.27 1.27)))
     )
@@
     (pin "3")
     (pin "4")
+    (pin "MP")
     (instances
       (project "Controller"
@@
     )
   )
-  (symbol (lib_id "power:GND") (at 139.7 162.56 0) (unit 1)
-    (in_bom yes) (on_board yes) (dnp no) (fields_autoplaced)
-    (property "Reference" "#PWR01" (at 139.7 168.91 0)
-      (effects (font (size 1.27 1.27)) hide)
-    )
-    (property "Value" "GND" (at 139.7 167.64 0)
-      (effects (font (size 1.27 1.27)))
-    )
-    (property "Footprint" "" (at 139.7 162.56 0)
-      (effects (font (size 1.27 1.27)) hide)
-    )
-    (property "Datasheet" "" (at 139.7 162.56 0)
+  (symbol (lib_id "power:GND") (at 139.7 165.1 0) (unit 1)
+    (in_bom yes) (on_board yes) (dnp no) (fields_autoplaced)
+    (property "Reference" "#PWR01" (at 139.7 171.45 0)
+      (effects (font (size 1.27 1.27)) hide)
+    )
+    (property "Value" "GND" (at 139.7 170.18 0)
+      (effects (font (size 1.27 1.27)))
+    )
+    (property "Footprint" "" (at 139.7 165.1 0)
+      (effects (font (size 1.27 1.27)) hide)
+    )
+    (property "Datasheet" "" (at 139.7 165.1 0)
       (effects (font (size 1.27 1.27)) hide)
     )
@@
     )
   )
-  (symbol (lib_id "power:GND") (at 173.99 109.22 0) (unit 1)
-    (in_bom yes) (on_board yes) (dnp no) (fields_autoplaced)
-    (property "Reference" "#PWR01" (at 173.99 115.57 0)
-      (effects (font (size 1.27 1.27)) hide)
-    )
-    (property "Value" "GND" (at 173.99 114.3 0)
-      (effects (font (size 1.27 1.27)))
-    )
-    (property "Footprint" "" (at 173.99 109.22 0)
-      (effects (font (size 1.27 1.27)) hide)
-    )
-    (property "Datasheet" "" (at 173.99 109.22 0)
+  (symbol (lib_id "power:GND") (at 173.99 111.76 0) (unit 1)
+    (in_bom yes) (on_board yes) (dnp no) (fields_autoplaced)
+    (property "Reference" "#PWR01" (at 173.99 118.11 0)
+      (effects (font (size 1.27 1.27)) hide)
+    )
+    (property "Value" "GND" (at 173.99 116.84 0)
+      (effects (font (size 1.27 1.27)))
+    )
+    (property "Footprint" "" (at 173.99 111.76 0)
+      (effects (font (size 1.27 1.27)) hide)
+    )
+    (property "Datasheet" "" (at 173.99 111.76 0)
       (effects (font (size 1.27 1.27)) hide)
     )
@@
   (symbol (lib_id "Connector_Generic:Conn_01x04") (at 146.05 158.75 0) (mirror x) (unit 1)
     (in_bom yes) (on_board yes) (dnp no)
-    (property "Reference" "J6" (at 146.05 163.83 0)
-      (effects (font (size 1.27 1.27)))
-    )
-    (property "Value" "QWIIC" (at 146.05 151.13 0)
+    (property "Reference" "J6" (at 146.05 151.13 0)
+      (effects (font (size 1.27 1.27)))
+    )
+    (property "Value" "QWIIC" (at 146.05 166.37 0)
       (effects (font (size 1.27 1.27)))
     )
@@
     (pin "3")
     (pin "4")
-    (instances
-      (project "Controller"
+    (pin "MP")
+    (instances
+      (project "Controller"

Commit message: BOM update
Parts:
- C2: DigiKey (none) -> 1276-2449-1-ND
- D14, D15, D16, D17, D18, D19, D20, D21: DigiKey D1213A-01WS-7 -> D1213A-01WS-7DICT-ND
- J1: DigiKey (none) -> 1175-1621-ND
- R24, R25, R26, R27, R28, R29: DigiKey (none) -> CR0805-FX-1002ELFCT-ND
Changed lines of the file:
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@@
+      (effects (font (size 1.27 1.27)) hide)
+    )
+    (property "DigiKey" "1276-2449-1-ND" (at 166.37 91.44 0)
       (effects (font (size 1.27 1.27)) hide)
     )
@@
       (effects (font (size 1.27 1.27)) hide)
     )
-    (property "DigiKey" "D1213A-01WS-7" (at 127 161.29 90)
+    (property "DigiKey" "D1213A-01WS-7DICT-ND" (at 127 161.29 90)
       (effects (font (size 1.27 1.27)) hide)
     )
@@
       (effects (font (size 1.27 1.27)) hide)
     )
+    (property "DigiKey" "CR0805-FX-1002ELFCT-ND" (at 115.57 41.91 0)
+      (effects (font (size 1.27 1.27)) hide)
+    )
     (pin "1")
     (pin "2")
@@
       (effects (font (size 1.27 1.27)) hide)
     )
+    (property "DigiKey" "CR0805-FX-1002ELFCT-ND" (at 115.57 95.25 0)
+      (effects (font (size 1.27 1.27)) hide)
+    )
     (pin "1")
     (pin "2")
@@
       (effects (font (size 1.27 1.27)) hide)
     )
+    (property "DigiKey" "CR0805-FX-1002ELFCT-ND" (at 128.27 41.91 0)
+      (effects (font (size 1.27 1.27)) hide)
+    )
     (pin "1")
     (pin "2")
@@
       (effects (font (size 1.27 1.27)) hide)
     )
-    (property "DigiKey" "D1213A-01WS-7" (at 148.59 107.95 90)
+    (property "DigiKey" "D1213A-01WS-7DICT-ND" (at 148.59 107.95 90)
       (effects (font (size 1.27 1.27)) hide)
     )
@@
       (effects (font (size 1.27 1.27)) hide)
     )
+    (property "DigiKey" "CR0805-FX-1002ELFCT-ND" (at 115.57 116.84 0)
+      (effects (font (size 1.27 1.27)) hide)
+    )
     (pin "1")
     (pin "2")
@@
       (effects (font (size 1.27 1.27)) hide)
     )
+    (property "DigiKey" "CR0805-FX-1002ELFCT-ND" (at 137.16 95.25 0)
+      (effects (font (size 1.27 1.27)) hide)
+    )
     (pin "1")
     (pin "2")
@@
       (effects (font (size 1.27 1.27)) hide)
     )
-    (property "DigiKey" "D1213A-01WS-7" (at 114.3 161.29 90)
+    (property "DigiKey" "D1213A-01WS-7DICT-ND" (at 114.3 161.29 90)
       (effects (font (size 1.27 1.27)) hide)
     )
@@
       (effects (font (size 1.27 1.27)) hide)
     )
-    (property "DigiKey" "D1213A-01WS-7" (at 140.97 59.69 90)
+    (property "DigiKey" "D1213A-01WS-7DICT-ND" (at 140.97 59.69 90)
       (effects (font (size 1.27 1.27)) hide)
     )
@@
       (effects (font (size 1.27 1.27)) hide)
     )
+    (property "DigiKey" "1276-2449-1-ND" (at 152.4 38.1 0)
+      (effects (font (size 1.27 1.27)) hide)
+    )
     (pin "1")
     (pin "2")
@@
       (effects (font (size 1.27 1.27)) hide)
     )
+    (property "DigiKey" "1276-2449-1-ND" (at 132.08 144.78 0)
+      (effects (font (size 1.27 1.27)) hide)
+    )
     (pin "1")
     (pin "2")
@@
       (effects (font (size 1.27 1.27)) hide)
     )
-    (property "DigiKey" "D1213A-01WS-7" (at 161.29 107.95 90)
+    (property "DigiKey" "D1213A-01WS-7DICT-ND" (at 161.29 107.95 90)
       (effects (font (size 1.27 1.27)) hide)
     )
@@
       (effects (font (size 1.27 1.27)) hide)
     )
-    (property "DigiKey" "D1213A-01WS-7" (at 128.27 59.69 90)
+    (property "DigiKey" "D1213A-01WS-7DICT-ND" (at 128.27 59.69 90)
       (effects (font (size 1.27 1.27)) hide)
     )
@@
       (effects (font (size 1.27 1.27)) hide)
     )
-    (property "DigiKey" "D1213A-01WS-7" (at 153.67 59.69 90)
+    (property "DigiKey" "D1213A-01WS-7DICT-ND" (at 153.67 59.69 90)
       (effects (font (size 1.27 1.27)) hide)
     )
@@
     )
     (property "Datasheet" "~" (at 166.37 49.53 0)
+      (effects (font (size 1.27 1.27)) hide)
+    )
+    (property "DigiKey" "1175-1621-ND" (at 166.37 49.53 0)
       (effects (font (size 1.27 1.27)) hide)
     )
@@
       (effects (font (size 1.27 1.27)) hide)
     )
+    (property "DigiKey" "CR0805-FX-1002ELFCT-ND" (at 137.16 116.84 0)
+      (effects (font (size 1.27 1.27)) hide)
+    )
     (pin "1")
     (pin "2")
@@
       (effects (font (size 1.27 1.27)) hide)
     )
-    (property "DigiKey" "D1213A-01WS-7" (at 115.57 59.69 90)
-      (effects (font (size 1.27 1.27)) hide)
-    )
+    (property "DigiKey" "D1213A-01WS-7DICT-ND" (at 115.57 59.69 90)
+      (effects (font (size 1.27 1.27)) hide)
+    )

Commit message: Schemas aktualisiert mit PDF
Other:
- company: (none) -> High5Dynamics
- title: (none) -> Controller
Changed lines of the file:
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@@
 (kicad_sch (version 20230121) (generator eeschema)
   (paper "A4")
+  (title_block
+    (title "Controller")
+    (date "2023-05-07")
+    (rev "1")
+    (company "High5Dynamics")
+  )
   (junction (at 127 156.21) (diameter 0) (color 0 0 0 0)
   )
