File: Controller/HW/KiCad_Files/USB_Programmer.kicad_sch (KiCad schematic)
At the start: 15 parts, among them J2 USB, Q1 Q_NPN_BEC, Q2 Q_NPN_BEC, U1 CP2102N-Axx-xQFN28, U2 USBLC6-2SC6

Commit message: PCB Zwischenstand
Parts:
- added D8: TX, LED_SMD:LED_0805_2012Metric, symbol Device:LED
- added D8: RX, LED_SMD:LED_0805_2012Metric, symbol Device:LED
- added R15 (x2): 1k, Resistor_SMD:R_0805_2012Metric, symbol Device:R
- J2: DigiKey (none) -> gfg
- Q1, Q2: value Q_NPN_BEC -> MMBT3904; DigiKey (none) -> 1727-4044-1-ND
- R6: value 10k -> 1k
- U1: DigiKey (none) -> 336-5890-1-ND
- U2: DigiKey (none) -> 497-5235-1-ND
Connections:
- net +3.3V: now also R15.1, R15.1
- net at U1.18 (~{RXT}/GPIO.1): now also D8.1 (K)
- net at U1.19 (~{TXT}/GPIO.0): now also D8.1 (K)
- new net: D8.2 (A), R15.2 (x2)
- no-connect marks 18 -> 16
Other:
- note added: "RX / TX LEDs"
- moved on the sheet: Q1, Q2, R10, R9

Commit message: BOM update
Parts:
- C2: DigiKey (none) -> 1276-2449-1-ND
- C3: DigiKey (none) -> 1276-1096-1-ND
- D8: DigiKey (none) -> 475-1410-1-ND
- J2: DigiKey gfg -> (none)
- R10, R7, R9: DigiKey (none) -> CR0805-FX-1002ELFCT-ND
- R11: DigiKey (none) -> CR0805-FX-2212ELFCT-ND
- R15, R6: DigiKey (none) -> CR0805-FX-1001ELFCT-ND
- R3, R4: DigiKey (none) -> CR0805-FX-5101ELFCT-ND
- R8: DigiKey (none) -> 311-47.5KCRCT-ND
Changed lines of the file:
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@@
+      (effects (font (size 1.27 1.27)) hide)
+    )
+    (property "DigiKey" "CR0805-FX-1002ELFCT-ND" (at 226.06 76.2 0)
       (effects (font (size 1.27 1.27)) hide)
     )
@@
       (effects (font (size 1.27 1.27)) hide)
     )
-    (property "DigiKey" "gfg" (at 60.96 93.98 0)
+    (property "DigiKey" "" (at 60.96 93.98 0)
       (effects (font (size 1.27 1.27)) hide)
     )
@@
       (effects (font (size 1.27 1.27)) hide)
     )
+    (property "DigiKey" "CR0805-FX-5101ELFCT-ND" (at 81.28 106.68 0)
+      (effects (font (size 1.27 1.27)) hide)
+    )
     (pin "1")
     (pin "2")
@@
       (effects (font (size 1.27 1.27)) hide)
     )
+    (property "DigiKey" "1276-1096-1-ND" (at 142.24 76.2 0)
+      (effects (font (size 1.27 1.27)) hide)
+    )
     (pin "1")
     (pin "2")
@@
       (effects (font (size 1.27 1.27)) hide)
     )
+    (property "DigiKey" "CR0805-FX-1002ELFCT-ND" (at 149.86 118.11 0)
+      (effects (font (size 1.27 1.27)) hide)
+    )
     (pin "1")
     (pin "2")
@@
     )
     (property "Datasheet" "~" (at 237.49 118.11 0)
+      (effects (font (size 1.27 1.27)) hide)
+    )
+    (property "DigiKey" "CR0805-FX-1001ELFCT-ND" (at 237.49 118.11 0)
       (effects (font (size 1.27 1.27)) hide)
     )
@@
       (effects (font (size 1.27 1.27)) hide)
     )
+    (property "DigiKey" "CR0805-FX-1002ELFCT-ND" (at 226.06 90.17 0)
+      (effects (font (size 1.27 1.27)) hide)
+    )
     (pin "1")
     (pin "2")
@@
       (effects (font (size 1.27 1.27)) hide)
     )
+    (property "DigiKey" "CR0805-FX-1001ELFCT-ND" (at 152.4 76.2 0)
+      (effects (font (size 1.27 1.27)) hide)
+    )
     (pin "1")
     (pin "2")
@@
     )
     (property "Datasheet" "~" (at 138.43 113.03 0)
+      (effects (font (size 1.27 1.27)) hide)
+    )
+    (property "DigiKey" "1276-2449-1-ND" (at 138.43 113.03 0)
       (effects (font (size 1.27 1.27)) hide)
     )
@@
       (effects (font (size 1.27 1.27)) hide)
     )
+    (property "DigiKey" "CR0805-FX-5101ELFCT-ND" (at 90.17 106.68 0)
+      (effects (font (size 1.27 1.27)) hide)
+    )
     (pin "1")
     (pin "2")
@@
       (effects (font (size 1.27 1.27)) hide)
     )
+    (property "DigiKey" "311-47.5KCRCT-ND" (at 128.27 113.03 0)
+      (effects (font (size 1.27 1.27)) hide)
+    )
     (pin "1")
     (pin "2")
@@
     )
     (property "Datasheet" "~" (at 223.52 127 0)
+      (effects (font (size 1.27 1.27)) hide)
+    )
+    (property "DigiKey" "475-1410-1-ND" (at 223.52 127 0)
       (effects (font (size 1.27 1.27)) hide)
     )
@@
       (effects (font (size 1.27 1.27)) hide)
     )
+    (property "DigiKey" "CR0805-FX-2212ELFCT-ND" (at 128.27 102.87 0)
+      (effects (font (size 1.27 1.27)) hide)
+    )
     (pin "1")
     (pin "2")
@@
       (effects (font (size 1.27 1.27)) hide)
     )
+    (property "DigiKey" "475-1410-1-ND" (at 237.49 127 0)
+      (effects (font (size 1.27 1.27)) hide)
+    )
     (pin "1")
     (pin "2")
@@
       (effects (font (size 1.27 1.27)) hide)
     )
+    (property "DigiKey" "CR0805-FX-1001ELFCT-ND" (at 223.52 118.11 0)
+      (effects (font (size 1.27 1.27)) hide)
+    )

Commit message: Schemas aktualisiert mit PDF
Other:
- company: (none) -> High5Dynamics
- title: (none) -> Controller
Changed lines of the file:
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@@
 (kicad_sch (version 20230121) (generator eeschema)
   (paper "A4")
+  (title_block
+    (title "Controller")
+    (date "2023-05-07")
+    (rev "1")
+    (company "High5Dynamics")
+  )
   (junction (at 138.43 107.95) (diameter 0) (color 0 0 0 0)
   )
